File: polarity-switch.kicad_sch (KiCad schematic)
At the start: 17 parts, among them U4 FDMQ8205A, U5 140356145400, U6 140356145400

Commit message: finished board
Other:
- moved on the sheet: D10, D11, D12, D13, D6, D7, R11, R12, R13, R14, R15, R16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

Commit message: production design files
Parts:
- D10, D11, D6, D7: Part Number (none) -> 1727-6235-1-ND
- D12, D13: Part Number (none) -> 1N4148WTDICT-ND
- U4: Part Number (none) -> FDMQ8205AOSCT-ND
- U5, U6: value 140356145400 -> ISOM8118DFHR; Part Number (none) -> 296-ISOM8118DFHRCT-ND
Changed lines of the file:
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@@
 			)
 		)
-		(property "Datasheet" "~"
+		(property "Datasheet" "https://www.diodes.com/assets/Datasheets/1N4148WT.pdf"
 			(at 189.23 101.6 0)
 			(effects
@@
 			)
 		)
-		(property "Part Number" ""
+		(property "Part Number" "1N4148WTDICT-ND"
 			(at 189.23 101.6 0)
 			(effects
@@
 					(size 1.27 1.27)
 				)
+				(hide yes)
 			)
 		)
@@
 					(size 1.27 1.27)
 				)
+				(hide yes)
 			)
 		)
@@
 					(size 1.27 1.27)
 				)
+				(hide yes)
 			)
 		)
@@
 			)
 		)
-		(property "Datasheet" "~"
+		(property "Datasheet" "https://assets.nexperia.com/documents/data-sheet/BZX585_SER.pdf"
 			(at 177.8 107.95 0)
 			(effects
@@
 			)
 		)
-		(property "Part Number" ""
+		(property "Part Number" "1727-6235-1-ND"
 			(at 177.8 107.95 0)
 			(effects
@@
 					(size 1.27 1.27)
 				)
+				(hide yes)
 			)
 		)
@@
 					(size 1.27 1.27)
 				)
+				(hide yes)
 			)
 		)
@@
 			)
 		)
-		(property "Datasheet" ""
+		(property "Datasheet" "https://www.onsemi.com/pdf/datasheet/fdmq8205a-d.pdf"
 			(at 152.4 99.06 0)
 			(effects
@@
 			)
 		)
-		(property "Part Number" ""
+		(property "Part Number" "FDMQ8205AOSCT-ND"
 			(at 152.4 99.06 0)
 			(effects
@@
 					(size 1.27 1.27)
 				)
+				(hide yes)
 			)
 		)
@@
 					(size 1.27 1.27)
 				)
+				(hide yes)
 			)
 		)
@@
 			)
 		)
-		(property "Datasheet" "~"
+		(property "Datasheet" "https://assets.nexperia.com/documents/data-sheet/BZX585_SER.pdf"
 			(at 127 107.95 0)
 			(effects
@@
 			)
 		)
-		(property "Part Number" ""
+		(property "Part Number" "1727-6235-1-ND"
 			(at 127 107.95 0)
 			(effects
@@
 					(size 1.27 1.27)
 				)
+				(hide yes)
 			)
 		)
@@
 			)
 		)
-		(property "Datasheet" "~"
+		(property "Datasheet" "https://assets.nexperia.com/documents/data-sheet/BZX585_SER.pdf"
 			(at 127 97.79 0)
 			(effects
@@
 			)
 		)
-		(property "Part Number" ""
+		(property "Part Number" "1727-6235-1-ND"
 			(at 127 97.79 0)
 			(effects
@@
 					(size 1.27 1.27)
 				)
+				(hide yes)
 			)
 		)
@@
 					(size 1.27 1.27)
 				)
+				(hide yes)
 			)
 		)
@@
 			)
 		)
-		(property "Datasheet" "~"
+		(property "Datasheet" "https://assets.nexperia.com/documents/data-sheet/BZX585_SER.pdf"
 			(at 177.8 97.79 0)
 			(effects
@@
 			)
 		)
-		(property "Part Number" ""
+		(property "Part Number" "1727-6235-1-ND"
 			(at 177.8 97.79 0)
 			(effects
@@
 					(size 1.27 1.27)
 				)
+				(hide yes)
 			)
 		)
@@
 					(size 1.27 1.27)
 				)
+				(hide yes)
 			)
 		)
@@
 					(size 1.27 1.27)
 				)
+				(hide yes)
 			)
 		)
@@
 			)
 		)
-		(property "Value" "140356145400"
+		(property "Value" "ISOM8118DFHR"
 			(at 93.98 97.79 0)
 			(effects
@@
 			)
 		)
-		(property "Datasheet" "https://www.we-online.com/components/media/o759429v6886%20Seriesdatasheet_WL-OCPT_SOP-4_SERIES_356_V2%20%28rev1%29.pdf"
+		(property "Datasheet" "https://www.ti.com/lit/ds/symlink/isom8111.pdf?ts=1741587314586&ref_url=https%253A%252F%252Fwww.ti.com%252Fproduct%252FISOM8111%253FkeyMatch%253DISOM8111%2526tisearch%253Duniversal_search%2526usecase%253DGPN-ALT"
 			(at 93.98 104.14 0)
 			(effects
@@
 			)
 		)
-		(property "Part Number" ""
+		(property "Part Number" "296-ISOM8118DFHRCT-ND"
 			(at 93.98 104.14 0)
 			(effects
@@
 					(size 1.27 1.27)
 				)
+				(hide yes)
 			)
 		)
@@
 			)
 		)
-		(property "Value" "140356145400"
+		(property "Value" "ISOM8118DFHR"
 			(at 210.82 97.79 0)
 			(effects
@@
 			)
 		)
-		(property "Datasheet" "https://www.we-online.com/components/media/o759429v6886%20Seriesdatasheet_WL-OCPT_SOP-4_SERIES_356_V2%20%28rev1%29.pdf"
+		(property "Datasheet" "https://www.ti.com/lit/ds/symlink/isom8111.pdf?ts=1741587314586&ref_url=https%253A%252F%252Fwww.ti.com%252Fproduct%252FISOM8111%253FkeyMatch%253DISOM8111%2526tisearch%253Duniversal_search%2526usecase%253DGPN-ALT"
 			(at 210.82 104.14 0)
 			(effects
@@
 			)
 		)
-		(property "Part Number" ""
+		(property "Part Number" "296-ISOM8118DFHRCT-ND"
 			(at 210.82 104.14 0)
 			(effects
@@
 					(size 1.27 1.27)
 				)
+				(hide yes)
 			)
 		)
@@
 					(size 1.27 1.27)
 				)
+				(hide yes)
 			)
 		)
@@
 			)
 		)
-		(property "Datasheet" "~"
+		(property "Datasheet" "https://www.diodes.com/assets/Datasheets/1N4148WT.pdf"
 			(at 115.57 101.6 0)
 			(effects
@@
 			)
 		)
-		(property "Part Number" ""
+		(property "Part Number" "1N4148WTDICT-ND"
 			(at 115.57 101.6 0)
 			(effects
@@
 					(size 1.27 1.27)
 				)
-			)
-		)
+				(hide yes)
+			)
+		)
