File: ECE2799_LED-Lamp.kicad_pcb (KiCad board)
At the start: 2 copper layers, 119 x 71 mm, 118 parts, among them J1 IEC_60320_C6_Receptacle, J2 Conn_01x04_MountingPin, J3 Conn_ARM_SWD_TagConnect_TC203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, J4 Conn_01x02_Pin, J5 Conn_01x04_MountingPin, J6 Conn_01x02, Q1 IGLR65R200D2, T1 750817251, U1 LT3799EMSE-PBF, U2 MP9989GV-Z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

Commit message: production design files
Parts:
- added H1: MountingHole_Pad, MountingHole:MountingHole_3.2mm_M3_Pad, F.Cu at (105.0, 90.0)
- added H2: MountingHole, MountingHole:MountingHole_3.2mm_M3, F.Cu at (189.0, 124.0)
- added H3: MountingHole, MountingHole:MountingHole_3.2mm_M3, F.Cu at (99.0, 135.0)
- added H4: MountingHole, MountingHole:MountingHole_3.2mm_M3, F.Cu at (99.0, 151.0)
- added H5: MountingHole, MountingHole:MountingHole_3.2mm_M3, F.Cu at (228.0, 135.0)
- added H6: MountingHole, MountingHole:MountingHole_3.2mm_M3, F.Cu at (228.0, 151.0)
- C23: value 1u -> 10u
- C8: footprint Capacitor_SMD:C_0805_2012Metric -> Capacitor_SMD:C_0603_1608Metric
- R1, R32: footprint Resistor_SMD:R_1812_4532Metric -> Resistor_SMD:R_2010_5025Metric
- U5, U6: value 140356145400 -> ISOM8118DFHR
- moved C18 10.0 mm to (210.0, 137.0)
- moved C19 10.0 mm to (212.0, 149.0)
- moved CS1 10.0 mm to (156.0, 139.0)
- moved G5 10.0 mm to (203.0, 143.0)
- moved J2 10.0 mm to (220.0, 143.0)
- moved JP3 10.0 mm to (217.0, 134.0)
- moved JP4 10.0 mm to (220.0, 134.0)
- moved R17 10.0 mm to (218.0, 138.0)
- moved R21 10.0 mm to (218.0, 148.0)
- moved R22 10.0 mm to (215.0, 133.0)
- moved R24 10.0 mm to (222.0, 133.0)
- moved U8 10.0 mm to (210.0, 143.0)
- moved R1 0.50 mm to (143.5, 89.5)
- moved R10 0.50 mm to (138.5, 93.5)
Routing:
- net GND: track 10.6 -> 14.7 mm
- net /DIR_A: track 6.33 -> 5.83 mm
Other:
- board size 119 x 71 mm -> 139 x 71 mm
- board text added: "${COMMENT1} ${COMMENT2} ${COMMENT3}"
- board text added: "${TITLE} v${REVISION} ${COMPANY} ${ISSUE_DATE}"

Commit message: board interconnects
Parts:
- added J7: Spade Terminal, 1212:1212, F.Cu at (112.5, 90.0)
- added J8: Spade Terminal, 1212:1212, F.Cu at (117.5, 90.0)
- D10, D11, D12, D13, D6, D7, R11, R13, R14, R9, U4: moved to B.Cu
- J6: value Conn_01x02 -> 2601-3102; footprint Connector_Wire:SolderWire-0.75sqmm_1x02_P4.8mm_D1.25mm_OD2.3mm -> KiCad:26013102
- moved R13 27.5 mm to (196.0, 119.0), turned to 0 degrees
- moved D13 25.2 mm to (196.0, 117.0), turned to 180 degrees
- moved D10 24.1 mm to (193.0, 119.0), turned to 90 degrees
- moved R14 23.0 mm to (196.0, 115.0), turned to 180 degrees
- moved D11 20.1 mm to (193.0, 115.0), turned to -90 degrees
- moved R12 18.2 mm to (196.0, 113.0), turned to 0 degrees
- moved U4 17.7 mm to (188.0, 117.0), turned to 0 degrees
- moved R11 16.6 mm to (180.0, 115.0), turned to 0 degrees
- moved D6 16.1 mm to (183.0, 119.0), turned to 90 degrees
- moved D12 15.8 mm to (180.0, 117.0), turned to 0 degrees
- moved D7 15.6 mm to (183.0, 115.0), turned to -90 degrees
- moved R9 15.6 mm to (180.0, 119.0), turned to 180 degrees
- moved R6 15.3 mm to (180.0, 113.0)
- moved U5 4.00 mm to (159.8, 124.0)
- moved U6 4.00 mm to (159.8, 128.0)
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Connections:
- J1 pad 1: /AC+ -> /AC_Input/AC+_in
- J6 pad 2: /LED_B -> /LED_A
Routing:
- net /DC-: track 96.3 -> 26.5 mm, vias 7 -> 17
- net /LED_B: track 6.86 -> 22.3 mm
- net /LED_A: track 6.86 -> 21.4 mm
- net /AC_Input/AC+_in: track 0.00 -> 14.3 mm
- net /AC+: track 32.9 -> 44.8 mm
- net Net-(D6-K): track 46.1 -> 38.4 mm
- net Net-(D10-K): track 53.8 -> 47.0 mm
- net +3V3: track 106.1 -> 99.3 mm
- net Net-(R15-Pad2): track 10.7 -> 7.00 mm
- net /DC+: track 19.4 -> 20.4 mm, vias 5 -> 22
- net Net-(R16-Pad1): track 10.2 -> 10.8 mm
- net GNDPWR: vias 73 -> 70
