File: mcu.kicad_sch (KiCad schematic)
At the start: 33 parts, among them J3 Conn_ARM_SWD_TagConnect_TC203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, J4 Conn_01x02_Pin, U7 RP2040, U9 AT25xxx, Y1 830070868

Commit message: sim and pdf
Other:
- note added: "PWM frequency = 1907 Hz"
Changed lines of the file:
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@@
 		(comment 3 "Bryan, Tahje")
+	)
+	(text "PWM frequency = 1907 Hz"
+		(exclude_from_sim no)
+		(at 195.834 87.122 0)
+		(effects
+			(font
+				(size 1.27 1.27)
+			)
+		)
 	)
 	(junction
