File: Touch/Touch.kicad_pcb (KiCad board)
At the start: 2 copper layers, 119 x 24 mm, 12 parts, among them J2 Conn_01x04_MountingPin, U8 CY8C20666A-24LQXI

Commit message: production design files
Parts:
- added H3: MountingHole, MountingHole:MountingHole_3.2mm_M3, F.Cu at (99.0, 135.0)
- added H4: MountingHole, MountingHole:MountingHole_3.2mm_M3, F.Cu at (99.0, 151.0)
- added H5: MountingHole, MountingHole:MountingHole_3.2mm_M3, F.Cu at (228.0, 135.0)
- added H6: MountingHole, MountingHole:MountingHole_3.2mm_M3, F.Cu at (228.0, 151.0)
- moved C18 10.0 mm to (210.0, 137.0)
- moved C19 10.0 mm to (212.0, 149.0)
- moved CS1 10.0 mm to (156.0, 139.0)
- moved G5 10.0 mm to (203.0, 143.0)
- moved J2 10.0 mm to (220.0, 143.0)
- moved JP3 10.0 mm to (217.0, 134.0)
- moved JP4 10.0 mm to (220.0, 134.0)
- moved R17 10.0 mm to (218.0, 138.0)
- moved R21 10.0 mm to (218.0, 148.0)
- moved R22 10.0 mm to (215.0, 133.0)
- moved R24 10.0 mm to (222.0, 133.0)
- moved U8 10.0 mm to (210.0, 143.0)
Other:
- board size 119 x 24 mm -> 139 x 24 mm
- board text added: "${COMMENT1} ${COMMENT2} ${COMMENT3}"
- board text added: "${TITLE} v${REVISION} ${COMPANY} ${ISSUE_DATE}"
