File: Touch/capacitive-touch.kicad_sch (KiCad schematic)
At the start: 11 parts, among them U8 CY8C20666A-24LQXI

Commit message: production design files
Parts:
- added H3, H4, H5, H6: MountingHole, MountingHole:MountingHole_3.2mm_M3, symbol Mechanical:MountingHole
